Commit message: robot urdf xacro more consistent

File: agilex_scout/urdf/mobile_robot/scout_v2.xacro (robot description, xacro)
@@ -15,14 +15,21 @@
 	<xacro:arg name="odometry_source" default="encoders" />
 	<xacro:property name="odometry_source" value="$(arg odometry_source)"/>
-	<link name="base_footprint">
+	<!-- virtual joints to link to ground and to odom -->
+	<link name="base_link">
 		<visual>
-			<origin xyz="0 0 0" rpy="0 0 0" />
+			<origin xyz="0 0 ${wheel_radius - wheel_vertical_offset}" rpy="0 0 0" />
 		</visual>
 	</link>
-    <joint name="base_footprint_to_base_link" type="fixed">
-        <origin xyz="0 0 ${wheel_radius - wheel_vertical_offset}" rpy="0 0 0" />
-        <parent link="base_footprint" />
-        <child link="mobile_robot_base_link" />
+    <joint name="base_link_to_base_footprint" type="fixed">
+        <origin xyz="0 0 ${- wheel_radius + wheel_vertical_offset}" rpy="0 0 0" />
+        <parent link="base_link" />
+        <child link="base_footprint" />
     </joint>
+	<link name="base_footprint"/>
+	<joint name="base_footprint_to_mobile_robot" type="fixed">
+		<origin xyz="0 0 ${wheel_radius - wheel_vertical_offset}" rpy="0 0 0" />
+		<parent link="base_footprint" />
+		<child link="mobile_robot_base_link" />
+	</joint>
 	<!-- Base link -->
 	<link name="mobile_robot_base_link">

Commit message: fix xacro tf tree

File: agilex_scout/urdf/mobile_robot/scout_v2.xacro (robot description, xacro)
@@ -14,22 +14,18 @@
 	<!-- odometry source: world ground truth or wheels encoders -->
 	<xacro:arg name="odometry_source" default="encoders" />
-	<xacro:property name="odometry_source" value="$(arg odometry_source)"/>
-    <!-- load gazebo xacro -->
-    <xacro:arg name="load_gazebo" default="true" />
+	<xacro:property name="odometry_source" value="$(arg odometry_source)" />
+	<!-- load gazebo xacro -->
+	<xacro:arg name="load_gazebo" default="true" />
 	<!-- virtual joints to link to ground and to odom -->
-	<link name="base_link">
-		<visual>
-			<origin xyz="0 0 ${wheel_radius - wheel_vertical_offset}" rpy="0 0 0" />
-		</visual>
-	</link>
-    <joint name="base_link_to_base_footprint" type="fixed">
-        <origin xyz="0 0 ${- wheel_radius + wheel_vertical_offset}" rpy="0 0 0" />
-        <parent link="base_link" />
-        <child link="base_footprint" />
-    </joint>
-	<link name="base_footprint"/>
-	<joint name="base_footprint_to_mobile_robot" type="fixed">
+	<link name="base_footprint" />
+	<joint name="base_footprint_to_base_link" type="fixed">
 		<origin xyz="0 0 ${wheel_radius - wheel_vertical_offset}" rpy="0 0 0" />
 		<parent link="base_footprint" />
+		<child link="base_link" />
+	</joint>
+	<link name="base_link" />
+	<joint name="base_link_to_mobile_robot" type="fixed">
+		<origin xyz="0 0 0" rpy="0 0 0" />
+		<parent link="base_link" />
 		<child link="mobile_robot_base_link" />
 	</joint>
@@ -39,5 +35,6 @@
 			<origin xyz="0 0 0" rpy="0 0 0" />
 			<geometry>
-				<mesh filename="file://$(find agilex_scout)/meshes/mobile_robot/mobile_robot_base_link.dae" />
+				<mesh
+					filename="file://$(find agilex_scout)/meshes/mobile_robot/mobile_robot_base_link.dae" />
 			</geometry>
 		</visual>
@@ -75,10 +72,12 @@
 	<!-- wheel labeled from 0 to 3, conter-clockwise, starting from front right wheel -->
 	<!-- motor 1 and 2 (left side) are mechanically installed in a reversed direction -->
-	<xacro:scout_wheel_type1 wheel_prefix="front_right" x="${wheelbase/2}" y="${-track/2}" z="${wheel_vertical_offset}"
-		phi="0" />
-	<xacro:scout_wheel_type2 wheel_prefix="front_left" x="${wheelbase/2}" y="${track/2}" z="${wheel_vertical_offset}" phi="0" />
-	<xacro:scout_wheel_type1 wheel_prefix="rear_left" x="${-wheelbase/2}" y="${track/2}" z="${wheel_vertical_offset}" phi="0" />
-	<xacro:scout_wheel_type2 wheel_prefix="rear_right" x="${-wheelbase/2}" y="${-track/2}" z="${wheel_vertical_offset}"
-		phi="0" />
+	<xacro:scout_wheel_type1 wheel_prefix="front_right" x="${wheelbase/2}" y="${-track/2}"
+		z="${wheel_vertical_offset}" phi="0" />
+	<xacro:scout_wheel_type2 wheel_prefix="front_left" x="${wheelbase/2}" y="${track/2}"
+		z="${wheel_vertical_offset}" phi="0" />
+	<xacro:scout_wheel_type1 wheel_prefix="rear_left" x="${-wheelbase/2}" y="${track/2}"
+		z="${wheel_vertical_offset}" phi="0" />
+	<xacro:scout_wheel_type2 wheel_prefix="rear_right" x="${-wheelbase/2}" y="${-track/2}"
+		z="${wheel_vertical_offset}" phi="0" />
 	<link name="front_mount" />
 	<joint name="front_mount_joint" type="fixed">
@@ -94,6 +93,6 @@
 	</joint>
 	<!-- Gazebo definitions  -->
-    <xacro:if value="$(arg load_gazebo)">
-	    <xacro:include filename="$(find agilex_scout)/urdf/mobile_robot/scout_v2.gazebo" />
-    </xacro:if>
+	<xacro:if value="$(arg load_gazebo)">
+		<xacro:include filename="$(find agilex_scout)/urdf/mobile_robot/scout_v2.gazebo" />
+	</xacro:if>
 </robot>

File: agilex_scout/urdf/mobile_robot/scout_wheel_type1.xacro (robot description, xacro)
@@ -60,11 +60,23 @@
 			</collision>
 		</link>
-		<joint name="${wheel_prefix}_wheel" type="continuous">
-			<parent link="mobile_robot_base_link" />
-			<child link="${wheel_prefix}_wheel_link" />
-			<origin xyz="${x} ${y} ${z}" rpy="${phi} 0.0 0.0" />
-			<axis xyz="0 1 0" rpy="0 0 0" />
-			<dynamics damping="0.0" friction="20" />
-		</joint>
+		<!-- if gazebo is loaded, simulate the robot wheel rotations and broadcast the join states-->
+		<xacro:if value="$(arg load_gazebo)">
+			<joint name="${wheel_prefix}_wheel" type="continuous">
+				<parent link="mobile_robot_base_link" />
+				<child link="${wheel_prefix}_wheel_link" />
+				<origin xyz="${x} ${y} ${z}" rpy="${phi} 0.0 0.0" />
+				<axis xyz="0 1 0" rpy="0 0 0" />
+				<dynamics damping="0.0" friction="20" />
+			</joint>
+		</xacro:if>
+		<!-- if real robot is loaded, fixed wheels are used because no joint broadcasters are available -->
+		<xacro:unless value="$(arg load_gazebo)">
+			<joint name="${wheel_prefix}_wheel" type="fixed">
+				<parent link="mobile_robot_base_link" />
+				<child link="${wheel_prefix}_wheel_link" />
+				<origin xyz="${x} ${y} ${z}" rpy="${phi} 0.0 0.0" />
+				<axis xyz="0 1 0" rpy="0 0 0" />
+			</joint>
+		</xacro:unless>
 	</xacro:macro>
 </robot>

File: agilex_scout/urdf/mobile_robot/scout_wheel_type2.xacro (robot description, xacro)
@@ -60,11 +60,23 @@
 			</collision>
 		</link>
-		<joint name="${wheel_prefix}_wheel" type="continuous">
-			<parent link="mobile_robot_base_link" />
-			<child link="${wheel_prefix}_wheel_link" />
-			<origin xyz="${x} ${y} ${z}" rpy="${phi} 0.0 0.0" />
-			<axis xyz="0 1 0" rpy="0 0 0" />
-			<dynamics damping="0.0" friction="20" />
-		</joint>
+		<!-- if gazebo is loaded, simulate the robot wheel rotations and broadcast the join states-->
+		<xacro:if value="$(arg load_gazebo)">
+			<joint name="${wheel_prefix}_wheel" type="continuous">
+				<parent link="mobile_robot_base_link" />
+				<child link="${wheel_prefix}_wheel_link" />
+				<origin xyz="${x} ${y} ${z}" rpy="${phi} 0.0 0.0" />
+				<axis xyz="0 1 0" rpy="0 0 0" />
+				<dynamics damping="0.0" friction="20" />
+			</joint>
+		</xacro:if>
+		<!-- if real robot is loaded, fixed wheels are used because no joint broadcasters are available -->
+		<xacro:unless value="$(arg load_gazebo)">
+			<joint name="${wheel_prefix}_wheel" type="fixed">
+				<parent link="mobile_robot_base_link" />
+				<child link="${wheel_prefix}_wheel_link" />
+				<origin xyz="${x} ${y} ${z}" rpy="${phi} 0.0 0.0" />
+				<axis xyz="0 1 0" rpy="0 0 0" />
+			</joint>
+		</xacro:unless>
 	</xacro:macro>
 </robot>

Commit message: navigation now working on real robot!

File: agilex_scout/urdf/mobile_robot/scout_v2.xacro (robot description, xacro)
@@ -57,5 +57,5 @@
 			<!-- <mass value="50" /> -->
 			<!-- <origin xyz="-0.00065 -0.085 0.062" />
-            <inertia ixx="0.6022" ixy="-0.02364" ixz="-0.1197" iyy="1.7386" iyz="-0.001544" izz="2.0296" /> -->
+			<inertia ixx="0.6022" ixy="-0.02364" ixz="-0.1197" iyy="1.7386" iyz="-0.001544" izz="2.0296" /> -->
 			<origin xyz="0.0 0.0 0.0" />
 			<inertia ixx="2.288641" ixy="0" ixz="0" iyy="5.103976" iyz="0" izz="3.431465" />
