Commit message: scout supports reverse motion, corrected lidar URDF and new map created

File: agilex_scout/urdf/robot.urdf.xacro (robot description, xacro)
@@ -12,6 +12,6 @@
 		<xacro:include filename="$(find agilex_scout)/urdf/sensors/os1.urdf" />
 		<joint name="os1_joint" type="fixed">
-			<origin xyz="0.15 0.0 0.49" rpy="0.0 0.0 0.0" />
-			<parent link="base_link" />
+			<origin xyz="0.2 0.0 0.64" rpy="0.0 0.0 0.0" />
+			<parent link="mobile_robot_base_link" />
 			<child link="os_sensor" />
 		</joint>

File: agilex_scout/urdf/sensors/os1.urdf (robot description, URDF)
Before this commit: robot os1_description, 1 links, 0 joints
Links:
- link os_sensor: geometry visual mesh filename=file://$(find agilex_scout)/meshes/sensors/laser_link.stl scale=1.0 1.0 1.0
